File: FrontPanel.kicad_sch (KiCad schematic)
At the start: 72 parts, among them J1 Screw_Terminal_01x03, Q1 TIP42, Q2 TIP42, Q3 TIP42, Q4 BC856, U1 LM321, U2 LM321, U3 MCP41U83x-xxxx-ST 5k, U4 MCP41U83x-xxxx-ST 100k, U5 MCP41U83x-xxxx-ST 100k, U6 MCP41U83x-xxxx-ST 5k

Commit message: many changes
Parts:
- removed C1, C2, C3, C4: 2200u, Capacitor_THT:CP_Radial_D18.0mm_P7.50mm, symbol Device:C_Polarized
- removed C12, C15, C16: 100n, Capacitor_SMD:C_1210_3225Metric_Pad1.33x2.70mm_HandSolder, symbol Device:C
- removed D1, D10, D11, D12, D13, D14, D15, D16, D2, D3, D4, D5, D6, D7, D8, D9: 1N5406, Diode_THT:D_DO-201AD_P15.24mm_Horizontal, symbol Diode:1N5406
- removed J1: Screw_Terminal_01x03, symbol Connector:Screw_Terminal_01x03
- removed Q1, Q2, Q3: TIP42, Package_TO_SOT_THT:TO-220-3_Vertical, symbol Transistor_BJT:TIP42
- removed R1, R10, R11, R12, R2, R3, R4, R5, R6, R7, R8, R9: 5mOhm, Resistor_SMD:R_Shunt_Vishay_WSK2512_6332Metric_T2.21mm, symbol Device:R_Shunt
- removed R21, R22: 1k, Resistor_SMD:R_1210_3225Metric_Pad1.30x2.65mm_HandSolder, symbol Device:R
- removed U3, U6: MCP41U83x-xxxx-ST 5k, Package_SO:TSSOP-14_4.4x5mm_P0.65mm, symbol Potentiometer_Digital:MCP41U83x-xxxx-ST
- removed U4, U5: MCP41U83x-xxxx-ST 100k, Package_SO:TSSOP-14_4.4x5mm_P0.65mm, symbol Potentiometer_Digital:MCP41U83x-xxxx-ST
- added C17, C30: 100n, Capacitor_SMD:C_1210_3225Metric_Pad1.33x2.70mm_HandSolder, symbol Device:C
- added C18: 2.2u, Capacitor_THT:CP_Radial_D18.0mm_P7.50mm, symbol Device:C_Polarized
- added Q3, Q5: IRF540N, Package_TO_SOT_SMD:TO-263-2, symbol Transistor_FET:IRF540N
- added R1, R2, R3, R4, R54: 5m, Resistor_SMD:R_0603_1608Metric_Pad0.98x0.95mm_HandSolder, symbol Device:R
- added R5, R56, R58, R59: 5.1k, Resistor_SMD:R_1210_3225Metric_Pad1.30x2.65mm_HandSolder, symbol Device:R
- added R51: 5m 333mW, Resistor_SMD:R_0603_1608Metric_Pad0.98x0.95mm_HandSolder, symbol Device:R
- added R6: 330, Resistor_SMD:R_1210_3225Metric_Pad1.30x2.65mm_HandSolder, symbol Device:R
- added R7: 10k, Resistor_SMD:R_1210_3225Metric_Pad1.30x2.65mm_HandSolder, symbol Device:R
- added RV10, RV11, RV9: 5k, Potentiometer_THT:Potentiometer_Bourns_3299W_Vertical, symbol Device:R_Potentiometer_Trim
- added TP10, TP11, TP12, TP13, TP14, TP3, TP8, TP9: TestPoint, TestPoint:TestPoint_Keystone_5019_Miniature, symbol Connector:TestPoint
- added U16: LM321, Package_SO:SSOP-14_5.3x6.2mm_P0.65mm, symbol Amplifier_Operational:LM321
- added U18: MCP3425Axx-xCH, Package_TO_SOT_SMD:SOT-23-6, symbol Analog_ADC:MCP3425Axx-xCH
- added U19, U3: OPA552U, Package_SO:SOIC-8_3.9x4.9mm_P1.27mm, symbol Amplifier_Operational:OPA552U
- added U20: Optocoupler_DC_PhotoNPN_AKEC, Package_DIP:DIP-4_W7.62mm_Socket_LongPads, symbol Isolator:Optocoupler_DC_PhotoNPN_AKEC
- added U4: LM4132xMF-3.3, Package_TO_SOT_SMD:SOT-23-5, symbol Reference_Voltage:LM4132xMF-3.3
- added U5, U7: DAC121C081CIMK, Package_TO_SOT_SMD:SOT-23-6, symbol Analog_DAC:DAC121C081CIMK
- C13, C5, C6, C7: footprint (none) -> Capacitor_THT:CP_Radial_D18.0mm_P7.50mm
Connections:
- net +5V: now also TP13.1, U4.4 (VIN); no longer C14.1, C7.1, R13.1, RV1.1, U1.5 (V+)
- net GND: now also C11.2, C14.2, C5.2, C6.2, C17.2, C18.2, C30.2, R54.1, RV10.3, RV11.3, RV9.1, RV9.2, TP8.1, U16.2 (V-), U16.3 (-), U18.2 (V_{SS}), U18.6 (Vin-), U19.1 (V-), U19.4 (V-), U19.5 (V-), U20.2, U3.1 (V-), U3.4 (V-), U3.5 (V-), U5.3 (GND), U5.6 (ADR0), U7.3 (GND); no longer D19.1 (K), D20.2 (A), R14.2, RV1.3, U1.2 (V-), U2.2 (V-)
- net at C10.2, R15.2: now also R58.2, U3.6
- net V_{OUT}: now reaches C11.1, C5.1, C6.1
- net V_{OUT}: now also C10.1, C13.2, D19.1 (K), D20.2 (A), R14.2, RV1.3, U1.2 (V-), U2.2 (V-), Q5.2 (D), R1.2, R2.2, R3.2, R4.2, R51.2, RV10.2, RV11.2, TP11.1, U19.2 (-), U3.2 (-), U4.2 (GND), U4.3 (EN); no longer H1.1
- net at JP1.2 (B), TP2.1: now also Q3.1 (G)
- net at C13.1, R19.2: now also R59.2, U19.6
- net at R20.2: now also Q3.3 (S), R1.1, R2.1, R3.1, R4.1, R51.1
- net -5V renamed V_{OUT}-5V
- net V_{OUT}-5V: now also R5.1, TP12.1
- removed net LV_NEUT: C10.1, C11.2, C13.2, C14.2, C5.2, C6.2, H2.1
- new net: R59.1, RV11.1
- new net: C14.1, C17.1, C18.1, U4.5 (VREF), U5.2 (VA), U7.2 (VA), U7.6 (ADR0)
- new net: R58.1, RV10.1
- new net: H1.1, Q5.3 (S)
- new net: U19.3 (+), U7.1 (VOUT)
- new net: U3.3 (+), U5.1 (VOUT)
- new net: R56.1, RV9.3
- new net: Q5.1 (G), R5.2, R7.1
- new net: R7.2, U20.3
- new net: R6.2, U20.1
- new net: R56.2, TP14.1, U16.4, U18.1 (Vin+)
- new net: H2.1, R54.2, U16.1 (+)
- new net +35VDC: Q3.2 (D), TP10.1
- new net +3V3: C30.1, TP3.1, U16.5 (V+), U18.5 (V_{DD})
- new net CC_{thermal}: U19.8 (Flag)
- new net CV_{thermal}: U3.8 (Flag)
- new net OE: R6.1
- new net SCL0: U18.3 (SCL), U5.5 (SCL), U7.5 (SCL)
- new net SDA0: U18.4 (SDA), U5.4 (SDA), U7.4 (SDA)
- new net V_{OUT}+5V: C7.1, R13.1, RV1.1, TP9.1, U1.5 (V+), U19.7 (V+), U20.4, U3.7 (V+)
- no-connect marks 4 -> 0
Other:
- note added: "5V LOGIC"
- note added: "Addr = 0110 1000 = 0x68 = 88"
- note added: "Addr = 1000110 = 0x46 = 70"
- note added: "Addr = 1000111 = 0x47 = 71"
- note added: "Current control feedback"
- note added: "I = 10A / 5 = 2A ea P = I^{2}R = 2^{2} * 5m = 200mW ea"
- note added: "I2C0 for PSU monitoring I2C1 for HMI"
- note added: "Trim RV9 so 3.300V at TP14 when DUT at 10A load st 0.333V = 1A 10A / 2^{16} = 0.15mA resolution"
- note added: "Voltage control feedback"
- note removed: "Current control input"
- note removed: "THIS PART DOESN'T MAKE SENSE - Should the signal be brought to GND?"
- note removed: "TODO: WTF IS THIS CONNECTED TO?"
- note removed: "Voltage control input"
- moved on the sheet: C10, C11, C13, C5, C6, C7, C8, C9, D17, D18, D19, JP1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

Commit message: do some work on the regulator boards
Parts:
- C13, C18, C6, C7: footprint Capacitor_THT:CP_Radial_D18.0mm_P7.50mm -> Capacitor_THT:CP_Radial_D5.0mm_P2.00mm
- C5: footprint Capacitor_THT:CP_Radial_D18.0mm_P7.50mm -> Capacitor_THT:CP_Radial_D8.0mm_P3.50mm

Commit message: kicad v10. many changes to invididual boards
Parts:
- added J10: Screw_Terminal_01x03, TerminalBlock_4Ucon:TerminalBlock_4Ucon_1x03_P3.50mm_Vertical, symbol Connector:Screw_Terminal_01x03
- added J9: Screw_Terminal_01x02, TerminalBlock_4Ucon:TerminalBlock_4Ucon_1x02_P3.50mm_Horizontal, symbol Connector:Screw_Terminal_01x02
- Q3, Q5: footprint Package_TO_SOT_SMD:TO-263-2 -> Package_TO_SOT_THT:TO-220-3_Vertical
- U16: footprint Package_SO:SSOP-14_5.3x6.2mm_P0.65mm -> Package_TO_SOT_SMD:SOT-23-5_HandSoldering
Connections:
- net +35VDC: now also J9.1 (Pin_1)
- net GND: now also J9.2 (Pin_2)
- net V_{OUT}: now also J10.2 (Pin_2)
- net V_{OUT}+5V: now also J10.3 (Pin_3)
- net V_{OUT}-5V: now also R5.2, J10.1 (Pin_1); no longer R5.1
- net at RV9.3: now also R56.2; no longer R56.1
- net at Q5.1 (G), R7.1: now also R5.1; no longer R5.2
- net at TP14.1, U16.4, U18.1 (Vin+): now also R56.1; no longer R56.2
Other:
- moved on the sheet: R54, R56

Commit message: interim commit
Parts:
- added H11, H12, H13, H14, H5, H6: 3.5mm, MountingHole:MountingHole_3mm_Pad, symbol Mechanical:MountingHole
