File: Lab PSU.kicad_pcb (KiCad board)
At the start: 2 copper layers, 180 x 200 mm, 199 parts, among them J1 Screw_Terminal_01x04, J2 Conn_01x04, J3 Conn_01x06, J4 Screw_Terminal_01x03, J5 Screw_Terminal_01x03, J6 Screw_Terminal_01x03, Q3 IRF540N, Q4 BC856, Q5 IRF540N, SW1 RotaryEncoder_Switch, SW2 RotaryEncoder_Switch, U1 LM321, U11 CH340G, U12 Optocoupler_DC_PhotoNPN_AKEC, U13 Optocoupler_DC_PhotoNPN_AKEC, U14 LM317_SOT-223, U15 LM337_SOT223, U16 LM321, U17 LM317_SOT-223, U18 MCP3425Axx-xCH, U19 OPA552U, U2 LM321, U20 Optocoupler_DC_PhotoNPN_AKEC, U3 OPA552U, U4 LM4132xMF-3.3, U5 DAC121C081CIMK, U6 MCP23018x-x-SO, U7 DAC121C081CIMK, U8 XIAO-RP2350-SMD, U9 Optocoupler_DC_PhotoNPN_AKEC, Y1 12MHz

Commit message: do some work on the regulator boards
Parts:
- added J7: Screw_Terminal_01x03, TerminalBlock_4Ucon:TerminalBlock_4Ucon_1x03_P3.50mm_Vertical, F.Cu at (28.0, -192.0)
- added J8: Screw_Terminal_01x02, TerminalBlock_4Ucon:TerminalBlock_4Ucon_1x02_P3.50mm_Horizontal, F.Cu at (93.0, -191.2)
- C13, C18, C27, C28, C35, C6, C7: footprint Capacitor_THT:CP_Radial_D18.0mm_P7.50mm -> Capacitor_THT:CP_Radial_D5.0mm_P2.00mm
- C29, C33, C34: footprint Capacitor_THT:CP_Radial_D18.0mm_P7.50mm -> Capacitor_THT:CP_Radial_D10.0mm_P5.00mm_P7.50mm
- C31, C32, C37: footprint Capacitor_THT:CP_Radial_D18.0mm_P7.50mm -> Capacitor_THT:CP_Radial_D6.3mm_P2.50mm
- C5: footprint Capacitor_THT:CP_Radial_D18.0mm_P7.50mm -> Capacitor_THT:CP_Radial_D8.0mm_P3.50mm
- TP4: value TestPoint -> SDA0
- TP5: value TestPoint -> SCL0
- TP6: value TestPoint -> SDA1
- TP7: value TestPoint -> SCL1
- moved U14 240.6 mm to (100.0, -107.0)
- moved RV2 232.7 mm to (118.1, -98.0)
- moved RV3 232.7 mm to (118.1, -90.3)
- moved J4 230.5 mm to (135.5, -192.0)
- moved U15 226.0 mm to (100.2, -83.0)
- moved C33 221.5 mm to (85.0, -101.5), turned to -90 degrees
- moved C36 204.7 mm to (140.0, -98.0)
- moved C34 201.4 mm to (85.0, -90.5), turned to -90 degrees
- moved C38 200.7 mm to (140.0, -89.0)
- moved C28 183.5 mm to (97.0, -98.0), turned to -90 degrees
- moved R50 179.2 mm to (124.0, -104.0)
- moved C32 177.0 mm to (130.0, -99.0), turned to -90 degrees
- moved C27 163.7 mm to (97.0, -92.0), turned to -90 degrees
- moved R47 161.8 mm to (111.0, -104.0)
- moved R49 157.3 mm to (124.0, -82.0)
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Connections:
- C38 pad 1: V_{OUT}-5V -> V_{OUT}
- C38 pad 2: V_{OUT} -> V_{OUT}-5V
- J2 pad 4: /HMI/SCL1 -> /HMI/SDA1
- J4 pad 1: unconnected-(J4-Pin_1-Pad1) -> V_{OUT}+5V
- J4 pad 2: unconnected-(J4-Pin_2-Pad2) -> V_{OUT}
- J4 pad 3: unconnected-(J4-Pin_3-Pad3) -> V_{OUT}-5V
- J6 pad 1: 230VAC -> Net-(J6-Pin_1)
- RV6 pad 1: /HMI/SCL1 -> /HMI/SDA1
- TP6 pad 1: /HMI/SCL1 -> /HMI/SDA1
- TR1 pad 1: 230VAC -> Net-(J6-Pin_1)
- TR2 pad 1: 230VAC -> Net-(J7-Pin_1)
- U6 pad 13: /HMI/SCL1 -> /HMI/SDA1
- U8 pad 5: /HMI/SCL1 -> /HMI/SDA1
- Y1 pad 2: Net-(Y1-G-Pad2) -> GNDD
- Y1 pad 4: Net-(Y1-G-Pad2) -> GNDD
Routing:
- net NEUT: track 0.00 -> 167.2 mm
- net GND: track 166.6 -> 0.00 mm, vias 0 -> 2
- net V_{OUT}+5V: track 0.00 -> 153.0 mm
- net Net-(D30-A): track 0.00 -> 140.8 mm
- net V_{OUT}-5V: track 0.00 -> 137.2 mm
- net Net-(J6-Pin_1): track 0.00 -> 70.6 mm
- net V_{OUT}: track 0.00 -> 65.0 mm
- net Net-(U14-ADJ): track 0.00 -> 51.6 mm, vias 0 -> 1
- net Net-(D24-K): track 0.00 -> 50.9 mm
- net +5V: track 47.4 -> 0.00 mm
- net Net-(U15-ADJ): track 0.00 -> 45.9 mm
- net Net-(TR2-Pad2): track 0.00 -> 36.0 mm
- net Net-(TR1-Pad2): track 0.00 -> 36.0 mm
- net V_{OUT}+9VAC: track 0.00 -> 35.7 mm
- net Net-(J7-Pin_1): track 0.00 -> 28.7 mm
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- added copper zone on F.Cu, net +5V
- added copper zone on B.Cu, net GND
- added copper zone on F.Cu, net V_{OUT}

Commit message: shrink regulator board a little
Parts:
- removed J5: Screw_Terminal_01x03, TerminalBlock_4Ucon:TerminalBlock_4Ucon_1x03_P3.50mm_Vertical
- removed R46: 330, Resistor_SMD:R_1210_3225Metric_Pad1.30x2.65mm_HandSolder
- removed U13: Optocoupler_DC_PhotoNPN_AKEC, Package_DIP:DIP-4_W7.62mm_Socket_LongPads
- added H10: 3.5mm, MountingHole:MountingHole_3mm_Pad, F.Cu at (50.0, -5.00)
- added H3: 3.5mm, MountingHole:MountingHole_3mm_Pad, F.Cu at (5.00, -70.0)
- added H4: 3.5mm, MountingHole:MountingHole_3mm_Pad, F.Cu at (5.00, -5.00)
- added H5: 3.5mm, MountingHole:MountingHole_3mm_Pad, F.Cu at (195.0, -70.0)
- added H6: 3.5mm, MountingHole:MountingHole_3mm_Pad, F.Cu at (195.0, -5.00)
- added H7: 3.5mm, MountingHole:MountingHole_3mm_Pad, F.Cu at (150.0, -70.0)
- added H8: 3.5mm, MountingHole:MountingHole_3mm_Pad, F.Cu at (150.0, -5.00)
- added H9: 3.5mm, MountingHole:MountingHole_3mm_Pad, F.Cu at (50.0, -70.0)
- moved C38 77.2 mm to (99.0, -154.4), turned to 90 degrees
- moved C36 75.4 mm to (90.0, -154.4), turned to 90 degrees
- moved R49 66.4 mm to (106.0, -145.9), turned to 90 degrees
- moved C31 66.1 mm to (98.0, -147.9), turned to 0 degrees
- moved C32 63.8 mm to (89.0, -147.9), turned to 0 degrees
- moved R50 57.2 mm to (84.0, -144.9), turned to 90 degrees
- moved R48 55.1 mm to (106.0, -136.9), turned to 90 degrees
- moved RV3 52.7 mm to (97.7, -138.9), turned to 90 degrees
- moved RV2 49.6 mm to (90.0, -138.9), turned to 90 degrees
- moved U15 47.2 mm to (106.0, -129.9), turned to 90 degrees
- moved R47 42.5 mm to (84.0, -136.9), turned to 90 degrees
- moved J4 41.0 mm to (107.5, -222.0), turned to 180 degrees
- moved J8 39.4 mm to (68.5, -222.0), turned to 0 degrees
- moved R55 36.4 mm to (88.5, -194.0)
- moved C27 34.7 mm to (96.0, -126.7), turned to 0 degrees
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Connections:
- J4 pad 1: V_{OUT}+5V -> V_{OUT}-5V
- J4 pad 3: V_{OUT}-5V -> V_{OUT}+5V
Routing:
- net V_{OUT}+5V: track 153.0 -> 125.8 mm
- net V_{OUT}-5V: track 137.2 -> 114.8 mm
- net Net-(D25-K): track 102.6 -> 87.3 mm
- net Net-(D30-A): track 140.8 -> 151.2 mm
- net Net-(U15-ADJ): track 45.9 -> 36.0 mm
- net Net-(U14-ADJ): track 51.6 -> 45.7 mm
- net Net-(U17-ADJ): track 42.1 -> 36.7 mm
- net V_{OUT}+9VAC: track 35.7 -> 39.2 mm
- net V_{OUT}-9VAC: track 28.3 -> 29.8 mm
- net Net-(D24-K): track 50.9 -> 49.5 mm
Other:
- board size 180 x 200 mm -> 200 x 230 mm

Commit message: kicad v10. many changes to invididual boards
Parts:
- added C45: 100n, Capacitor_SMD:C_1210_3225Metric_Pad1.33x2.70mm_HandSolder, F.Cu at (82.5, -56.0)
- added J10: Screw_Terminal_01x03, TerminalBlock_4Ucon:TerminalBlock_4Ucon_1x03_P3.50mm_Vertical, B.Cu at (25.5, -6.92)
- added J11: Screw_Terminal_01x03, TerminalBlock_4Ucon:TerminalBlock_4Ucon_1x03_P3.50mm_Vertical, F.Cu at (270.5, -212.5)
- added J5: Screw_Terminal_01x02, TerminalBlock_4Ucon:TerminalBlock_4Ucon_1x02_P3.50mm_Horizontal, F.Cu at (251.5, -322.8)
- added J9: Screw_Terminal_01x02, TerminalBlock_4Ucon:TerminalBlock_4Ucon_1x02_P3.50mm_Horizontal, B.Cu at (189.5, -207.5)
- LED1, LED2, LED3, LED4, LED5, LED6: footprint PCM_marbastlib-various:LED_6028R -> PCM_marbastlib-mx:LED_MX_6028R; moved to B.Cu
- Q3, Q5: footprint Package_TO_SOT_SMD:TO-263-2 -> Package_TO_SOT_THT:TO-220-3_Vertical
- RV4, RV5, RV6, RV7, RV9, U8: moved to B.Cu
- U16: footprint Package_SO:SSOP-14_5.3x6.2mm_P0.65mm -> Package_TO_SOT_SMD:SOT-23-5_HandSoldering
- moved D16 480.3 mm to (222.6, -281.2), turned to 180 degrees
- moved D15 468.6 mm to (222.6, -274.5), turned to 180 degrees
- moved D12 467.3 mm to (242.6, -281.2), turned to 180 degrees
- moved D8 467.1 mm to (242.6, -308.0), turned to 180 degrees
- moved D14 456.9 mm to (222.6, -267.8), turned to 180 degrees
- moved D11 455.9 mm to (242.6, -274.5), turned to 180 degrees
- moved D7 455.7 mm to (242.6, -301.2), turned to 180 degrees
- moved D13 445.3 mm to (222.6, -261.0), turned to 180 degrees
- moved D10 444.7 mm to (242.6, -267.8), turned to 180 degrees
- moved D6 444.5 mm to (242.6, -294.5), turned to 180 degrees
- moved R7 433.7 mm to (238.0, -235.5)
- moved D9 433.6 mm to (242.6, -261.0), turned to 180 degrees
- moved D4 433.5 mm to (222.6, -308.0), turned to 180 degrees
- moved D5 433.4 mm to (242.6, -287.8), turned to 180 degrees
- moved R5 430.1 mm to (238.0, -240.0)
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Connections:
- C15 pad 1: /HMI/encSetB -> GND
- C15 pad 2: GND -> /HMI/encSetB
- C16 pad 1: /HMI/encSetA -> GND
- C16 pad 2: GND -> /HMI/encSetA
- C19 pad 1: /HMI/encSetS -> GND
- C19 pad 2: GND -> /HMI/encSetS
- C40 pad 1: /HMI/btnV_{lim} -> GND
- C40 pad 2: GND -> /HMI/btnV_{lim}
- C42 pad 1: /HMI/btnCancel -> GND
- C42 pad 2: GND -> /HMI/btnCancel
- C43 pad 1: /HMI/btnI_{lim} -> GND
- C43 pad 2: GND -> /HMI/btnI_{lim}
- J2 pad 2: V_{OUT}+5V -> +3V3
- R16 pad 1: /HMI/encSetB -> Net-(R16-Pad1)
- R16 pad 2: Net-(R16-Pad2) -> /HMI/encSetB
- R17 pad 1: /HMI/encSetA -> Net-(R17-Pad1)
- R17 pad 2: Net-(R17-Pad2) -> /HMI/encSetA
- R18 pad 1: Net-(R17-Pad2) -> +3V3
- R18 pad 2: +3V3 -> Net-(R17-Pad1)
- R23 pad 1: Net-(R16-Pad2) -> +3V3
- R23 pad 2: +3V3 -> Net-(R16-Pad1)
- R24 pad 1: Net-(R24-Pad1) -> +3V3
- R24 pad 2: +3V3 -> Net-(R24-Pad2)
- R25 pad 1: Net-(R24-Pad1) -> Net-(R24-Pad2)
- R35 pad 1: Net-(MX4-Pad2) -> /HMI/btnCV
- R35 pad 2: /HMI/btnCV -> Net-(MX4-Pad2)
- R36 pad 1: Net-(MX5-Pad2) -> /HMI/btnCC
- R36 pad 2: /HMI/btnCC -> Net-(MX5-Pad2)
- R37 pad 1: Net-(MX6-Pad2) -> /HMI/btnOE
- R37 pad 2: /HMI/btnOE -> Net-(MX6-Pad2)
- R5 pad 1: V_{OUT}-5V -> Net-(Q5-G)
- R5 pad 2: Net-(Q5-G) -> V_{OUT}-5V
- R56 pad 1: Net-(R56-Pad1) -> Net-(U18-Vin+)
- R56 pad 2: Net-(U18-Vin+) -> Net-(R56-Pad2)
- R8 pad 1: +3V3 -> Net-(U6-~{RESET})
- R8 pad 2: Net-(U6-~{RESET}) -> +3V3
- R9 pad 1: GND -> Net-(U6-ADDR)
- R9 pad 2: Net-(U6-ADDR) -> GND
- RV9 pad 3: Net-(R56-Pad1) -> Net-(R56-Pad2)
- SW1 pad A: Net-(R17-Pad2) -> Net-(R17-Pad1)
- SW1 pad B: Net-(R16-Pad2) -> Net-(R16-Pad1)
- SW1 pad S1: Net-(R24-Pad1) -> Net-(R24-Pad2)
- U6 pad 3: /HMI/btnCancel -> /HMI/btnV_{lim}
- U6 pad 4: /HMI/btnV_{lim} -> /HMI/btnI_{lim}
- U6 pad 5: /HMI/btnI_{lim} -> /HMI/btnCancel
- U8 pad 14: +5V -> unconnected-(U8-5V-Pad14)
Routing:
- net /HMI/SCL1: track 0.00 -> 146.0 mm, vias 0 -> 1
- net /FrontPanel/SCL0: track 0.00 -> 128.5 mm
- net /FrontPanel/SDA0: track 0.00 -> 128.3 mm
- net /HMI/SDA1: track 0.00 -> 109.4 mm
- net /HMI/btnCV: track 0.00 -> 105.7 mm, vias 0 -> 2
- net /HMI/encSetA: track 0.00 -> 94.6 mm, vias 0 -> 2
- net /HMI/encSetB: track 0.00 -> 89.5 mm, vias 0 -> 2
- net /HMI/encSetS: track 0.00 -> 84.5 mm, vias 0 -> 2
- net /HMI/btnCC: track 0.00 -> 80.8 mm, vias 0 -> 2
- net /HMI/btnCancel: track 0.00 -> 70.1 mm, vias 0 -> 2
- net V_{OUT}: track 65.0 -> 129.7 mm
- net /HMI/btnI_{lim}: track 0.00 -> 55.5 mm, vias 0 -> 2
- net /HMI/muxIntB: track 0.00 -> 54.8 mm, vias 0 -> 1
- net Net-(Q5-G): track 0.00 -> 54.1 mm
- net V_{OUT}-5V: track 114.8 -> 167.7 mm
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- added copper zone on F.Cu, net +25VAC
- added copper zone on F.Cu, net +35VDC
- added copper zone on F.Cu, net +3V3
- added copper zone on F.Cu, net 0VAC
Other:
- board size 200 x 230 mm -> 275 x 330 mm

Commit message: interim commit
Parts:
- added H11: 3.5mm, MountingHole:MountingHole_3mm_Pad, F.Cu at (67.5, -255.0)
- added H12: 3.5mm, MountingHole:MountingHole_3mm_Pad, F.Cu at (67.5, -135.0)
- added H13: 3.5mm, MountingHole:MountingHole_3mm_Pad, F.Cu at (130.0, -255.0)
- added H14: 3.5mm, MountingHole:MountingHole_3mm_Pad, F.Cu at (130.0, -135.0)
- added J12: Conn_01x20, Connector_PinSocket_2.54mm:PinSocket_1x20_P2.54mm_Vertical, F.Cu at (40.0, -147.1)
- added J13: Conn_01x20, Connector_PinSocket_2.54mm:PinSocket_1x20_P2.54mm_Vertical, F.Cu at (40.0, -144.5)
- added J14: Conn_01x20, Connector_PinSocket_2.54mm:PinSocket_1x20_P2.54mm_Vertical, F.Cu at (40.0, -142.0)
- added J15: Conn_01x20, Connector_PinSocket_2.54mm:PinSocket_1x20_P2.54mm_Vertical, F.Cu at (167.6, -205.7)
- added J16: Conn_01x20, Connector_PinSocket_2.54mm:PinSocket_1x20_P2.54mm_Vertical, F.Cu at (172.2, -205.7)
- added J17: Conn_01x20, Connector_PinSocket_2.54mm:PinSocket_1x20_P2.54mm_Vertical, F.Cu at (190.0, -314.2)
- added J18: Conn_01x20, Connector_PinSocket_2.54mm:PinSocket_1x20_P2.54mm_Vertical, F.Cu at (194.3, -314.2)
- added J19: Conn_01x20, Connector_PinHeader_2.54mm:PinHeader_1x20_P2.54mm_Vertical, F.Cu at (123.0, -390.0)
- added J20: Conn_01x20, Connector_PinHeader_2.54mm:PinHeader_1x20_P2.54mm_Vertical, F.Cu at (120.5, -390.0)
- moved R27 525.9 mm to (-240.7, -314.5)
- moved R43 525.9 mm to (-228.8, -314.5)
- moved C10 525.9 mm to (-274.9, -261.1)
- moved C13 525.9 mm to (-162.5, -316.8)
- moved C14 525.9 mm to (-274.9, -252.6)
- moved C17 525.9 mm to (-274.9, -248.3)
- moved C18 525.9 mm to (-162.5, -297.3)
- moved C20 525.9 mm to (-285.7, -288.6)
- moved C21 525.9 mm to (-285.7, -284.3)
- moved C22 525.9 mm to (-285.7, -280.1)
- moved C23 525.9 mm to (-285.7, -275.8)
- moved C24 525.9 mm to (-279.7, -288.6)
- moved C25 525.9 mm to (-279.7, -284.3)
- moved C26 525.9 mm to (-279.7, -280.1)
- moved C30 525.9 mm to (-274.9, -244.1)
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Connections:
- D27 pad 2: GND -> Net-(D27-A)
- D28 pad 1: GND -> Net-(D27-A)
- J4 pad 1: V_{OUT}-5V -> unconnected-(J4-Pin_1-Pad1)
- J4 pad 2: V_{OUT} -> unconnected-(J4-Pin_2-Pad2)
- J4 pad 3: V_{OUT}+5V -> unconnected-(J4-Pin_3-Pad3)
- TR2 pad 5: GND -> Net-(D27-A)
- TR2 pad 7: GND -> Net-(D27-A)
Routing:
- net unconnected-(J4-Pin_2-Pad2): track 0.00 -> 65.0 mm
- net Net-(Q5-G): track 54.1 -> 21.7 mm
- net V_{OUT}: track 129.7 -> 135.5 mm
Other:
- board size 275 x 330 mm -> 135 x 430 mm
